Commit message: Add files via upload

File: wheely_description/urdf/wheely.xacro (robot description, xacro)
@@ -24,47 +24,7 @@
   </collision>
 </link>
-<link name="left_wheel_v1_1">
+<link name="LIDAR_1">
   <inertial>
-    <origin rpy="0 0 0" xyz="-1.155962481396124e-17 0.012499999999999983 0.02500000000000005"/>
-    <mass value="0.18260507298990675"/>
-    <inertia ixx="0.000124" ixy="0.0" ixz="-0.0" iyy="0.000228" iyz="0.0" izz="0.000124"/>
-  </inertial>
-  <visual>
-    <origin rpy="0 0 0" xyz="0.0 -0.075 -0.025"/>
-    <geometry>
-      <mesh filename="package://wheely_description/meshes/left_wheel_v1_1.stl" scale="0.001 0.001 0.001"/>
-    </geometry>
-    <material name="rubber_soft"/>
-  </visual>
-  <collision>
-    <origin rpy="0 0 0" xyz="0.0 -0.075 -0.025"/>
-    <geometry>
-      <mesh filename="package://wheely_description/meshes/left_wheel_v1_1.stl" scale="0.001 0.001 0.001"/>
-    </geometry>
-  </collision>
-</link>
-<link name="right_wheel_v4_1">
-  <inertial>
-    <origin rpy="0 0 0" xyz="3.041195611585529e-18 -0.012500000000000039 0.025000000000000015"/>
-    <mass value="0.18260507298990675"/>
-    <inertia ixx="0.000124" ixy="0.0" ixz="-0.0" iyy="0.000228" iyz="0.0" izz="0.000124"/>
-  </inertial>
-  <visual>
-    <origin rpy="0 0 0" xyz="-0.0 0.075 -0.025"/>
-    <geometry>
-      <mesh filename="package://wheely_description/meshes/right_wheel_v4_1.stl" scale="0.001 0.001 0.001"/>
-    </geometry>
-    <material name="rubber_soft"/>
-  </visual>
-  <collision>
-    <origin rpy="0 0 0" xyz="-0.0 0.075 -0.025"/>
-    <geometry>
-      <mesh filename="package://wheely_description/meshes/right_wheel_v4_1.stl" scale="0.001 0.001 0.001"/>
-    </geometry>
-  </collision>
-</link>
-<link name="LIDAR_v3_1">
-  <inertial>
-    <origin rpy="0 0 0" xyz="1.6544549134691587e-18 -2.13153915195747e-17 0.010995989304812812"/>
+    <origin rpy="0 0 0" xyz="-3.226802273235357e-17 -2.1315391519574705e-17 0.010995989304812812"/>
     <mass value="0.046998226097703315"/>
     <inertia ixx="8e-06" ixy="-0.0" ixz="0.0" iyy="8e-06" iyz="0.0" izz="1.2e-05"/>
@@ -73,5 +33,5 @@
     <origin rpy="0 0 0" xyz="-0.0 0.0 -0.1"/>
     <geometry>
-      <mesh filename="package://wheely_description/meshes/LIDAR_v3_1.stl" scale="0.001 0.001 0.001"/>
+      <mesh filename="package://wheely_description/meshes/LIDAR_1.stl" scale="0.001 0.001 0.001"/>
     </geometry>
     <material name="plastic_glossy_grey"/>
@@ -80,25 +40,65 @@
     <origin rpy="0 0 0" xyz="-0.0 0.0 -0.1"/>
     <geometry>
-      <mesh filename="package://wheely_description/meshes/LIDAR_v3_1.stl" scale="0.001 0.001 0.001"/>
+      <mesh filename="package://wheely_description/meshes/LIDAR_1.stl" scale="0.001 0.001 0.001"/>
     </geometry>
   </collision>
 </link>
-<joint name="left_drive" type="continuous">
-  <origin rpy="0 0 0" xyz="0.0 0.075 0.025"/>
-  <parent link="base_link"/>
-  <child link="left_wheel_v1_1"/>
-  <axis xyz="0.0 -1.0 -0.0"/>
-</joint>
-<joint name="right_drive" type="continuous">
-  <origin rpy="0 0 0" xyz="0.0 -0.075 0.025"/>
-  <parent link="base_link"/>
-  <child link="right_wheel_v4_1"/>
-  <axis xyz="0.0 -1.0 -0.0"/>
-</joint>
+<link name="right_wheel_1">
+  <inertial>
+    <origin rpy="0 0 0" xyz="1.5103871126513457e-18 -0.01250000000000008 1.3877787807814457e-17"/>
+    <mass value="0.18260507298990675"/>
+    <inertia ixx="0.000124" ixy="0.0" ixz="-0.0" iyy="0.000228" iyz="-0.0" izz="0.000124"/>
+  </inertial>
+  <visual>
+    <origin rpy="0 0 0" xyz="-0.0 0.075 -0.05"/>
+    <geometry>
+      <mesh filename="package://wheely_description/meshes/right_wheel_1.stl" scale="0.001 0.001 0.001"/>
+    </geometry>
+    <material name="rubber_soft"/>
+  </visual>
+  <collision>
+    <origin rpy="0 0 0" xyz="-0.0 0.075 -0.05"/>
+    <geometry>
+      <mesh filename="package://wheely_description/meshes/right_wheel_1.stl" scale="0.001 0.001 0.001"/>
+    </geometry>
+  </collision>
+</link>
+<link name="left_wheel_1">
+  <inertial>
+    <origin rpy="0 0 0" xyz="-1.3090433312895435e-17 0.012499999999999983 3.469446951953614e-17"/>
+    <mass value="0.18260507298990675"/>
+    <inertia ixx="0.000124" ixy="0.0" ixz="-0.0" iyy="0.000228" iyz="0.0" izz="0.000124"/>
+  </inertial>
+  <visual>
+    <origin rpy="0 0 0" xyz="0.0 -0.075 -0.05"/>
+    <geometry>
+      <mesh filename="package://wheely_description/meshes/left_wheel_1.stl" scale="0.001 0.001 0.001"/>
+    </geometry>
+    <material name="rubber_soft"/>
+  </visual>
+  <collision>
+    <origin rpy="0 0 0" xyz="0.0 -0.075 -0.05"/>
+    <geometry>
+      <mesh filename="package://wheely_description/meshes/left_wheel_1.stl" scale="0.001 0.001 0.001"/>
+    </geometry>
+  </collision>
+</link>
 <joint name="lidar_rot" type="continuous">
   <origin rpy="0 0 0" xyz="0.0 0.0 0.1"/>
   <parent link="base_link"/>
-  <child link="LIDAR_v3_1"/>
+  <child link="LIDAR_1"/>
   <axis xyz="0.0 -0.0 1.0"/>
 </joint>
+<joint name="right_drive" type="continuous">
+  <origin rpy="0 0 0" xyz="0.0 -0.075 0.05"/>
+  <parent link="base_link"/>
+  <child link="right_wheel_1"/>
+  <axis xyz="0.0 -1.0 -0.0"/>
+</joint>
+<joint name="left_drive" type="continuous">
+  <origin rpy="0 0 0" xyz="0.0 0.075 0.05"/>
+  <parent link="base_link"/>
+  <child link="left_wheel_1"/>
+  <axis xyz="-0.0 1.0 0.0"/>
+</joint>
 </robot>
